File: hardware/DALI_USB.kicad_sch (KiCad schematic)
At the start: 4 parts

Commit message: second commit
Parts:
- removed H3, H4: 3.5, MountingHole:MountingHole_3.5mm, symbol Mechanical:MountingHole
Other:
- note added: "October 10, 2022"
