File: hardware/controller.kicad_sch (KiCad schematic)
At the start: 23 parts, among them J1 Tag_Connect, U2 STM32F091CCT6, Y1 8MHz

Commit message: second commit
Parts:
- removed C10: 1u, Capacitor_SMD:C_0603_1608Metric, symbol Device:C_Small
- removed C11: 10n, Capacitor_SMD:C_0603_1608Metric, symbol Device:C_Small
- removed C9: 100n, Capacitor_SMD:C_0603_1608Metric, symbol Device:C_Small
- removed FB1: 300R @ 100 MHz, Resistor_SMD:R_0603_1608Metric, symbol Device:Ferrite_Bead_Small
- removed R1: 0R, Resistor_SMD:R_0603_1608Metric, symbol Device:R_Small
- removed R2: 390R, Resistor_SMD:R_0603_1608Metric, symbol Device:R_Small
- removed R5: 1k, Resistor_SMD:R_0603_1608Metric, symbol Device:R_Small
- removed U2: STM32F091CCT6, Package_QFP:LQFP-48_7x7mm_P0.5mm, symbol MCU_ST_STM32F0:STM32F091CCTx
- removed Y1: 8MHz, Crystal:Crystal_SMD_5032-2Pin_5.0x3.2mm, symbol Device:Crystal_Small
- added U2: LPC1114FBD48-333, Package_QFP:LQFP-48_7x7mm_P0.5mm, symbol MCU_NXP_LPC:LPC1114FBD48-302
- added Y1: 12MHz, Crystal:Crystal_SMD_TXC_7M-4Pin_3.2x2.5mm, symbol Device:Crystal_GND24
- C6, C7: value 20p -> 18p; LCSC C1648 -> C38523
- R3, R4, R6: value 390R -> 120R; LCSC C23151 -> C114640
Connections:
- net +3V3: now also U2.44 (VDD), U2.8 (VDD)
- net DALI_RX: now also U2.33 (PIO1_0)
- net DALI_TX: now also U2.32 (PIO0_11)
- net GND: now also U2.41 (VSS), U2.5 (VSS), Y1.2, Y1.4
- net LED_DALI: now also U2.19 (PIO2_4)
- net LED_RX: now also U2.20 (PIO2_5)
- net LED_TX: now also U2.1 (PIO2_6)
- net OSC_IN: now also C6.1, U2.6 (XTALIN), Y1.1
- net OSC_OUT: now also C7.1, U2.7 (XTALOUT), Y1.3
- net SWCLK: now also U2.29 (PIO0_10)
- net SWDIO: now also U2.39 (PIO1_3)
- net UART_RX: now also U2.46 (PIO1_6)
- net UART_TX: now also U2.47 (PIO1_7)
- net \RESET: now also U2.3 (PIO0_0)
- no-connect marks 27 -> 33
Other:
- note added: "11. October 2022"
- moved on the sheet: C4, C5, C7, C8, D1, R3, R4, R6
