File: hardware/dali_phy.kicad_sch (KiCad schematic)
At the start: 14 parts, among them J2 2604-1102, Q1 MMBT2222A, Q2 MMBF4391, U3 LTV-357T, U4 LTV-357T

Commit message: second commit
Parts:
- D4: LCSC C90848 -> C90848
- R9: value 10k -> 5k1; LCSC C25804 -> C365441
Other:
- moved on the sheet: R9
