File: hardware/usb.kicad_sch (KiCad schematic)
At the start: 9 parts, among them J3 USB_B_Micro, U5 FT230XS

Commit message: second commit
Parts:
- removed J3: USB_B_Micro, DALI_USB V0:USB_Micro-B_XNJ, symbol Connector:USB_B_Micro
- added J3: USB_C_Receptacle_USB2.0, Connector_USB:USB_C_Receptacle_XKB_U262-16XN-4BVC11, symbol Connector:USB_C_Receptacle_USB2.0
- added R1, R2: 5k1, Resistor_SMD:R_0603_1608Metric, symbol Device:R
Connections:
- net GND: now also J3.A1 (GND), J3.A12 (GND), J3.B1 (GND), J3.B12 (GND), J3.S1 (SHIELD), R1.1, R2.2
- net at C15.1, FB2.2: now also J3.A4 (VBUS), J3.A9 (VBUS), J3.B4 (VBUS), J3.B9 (VBUS)
- net at R13.2: now also J3.A7 (D-), J3.B7 (D-)
- net at R14.2: now also J3.A6 (D+), J3.B6 (D+)
- new net: J3.B5 (CC2), R1.2
- new net: J3.A5 (CC1), R2.1
- no-connect marks 7 -> 8
Other:
- note added: "11. October 2022"
- moved on the sheet: C13, C14, C15, C16, FB2, R13, R14, U5
